Commit message: Models and launch file added

File: models/urdf/checkpoint.xacro (robot description, xacro)
@@ -3,4 +3,5 @@
   <xacro:arg name="mass" default="100" />
   <xacro:arg name="radius" default="0.75" />
+  <xacro:arg name="yaw" default="0.0" />
   <xacro:arg name="thickness" default="0.05" />
   <xacro:arg name="altitude" default="1.5" />
@@ -10,5 +11,5 @@
   <xacro:property name="scale_t" value="${$(arg thickness)/50}" />
   <xacro:property name="pillar_length" value="${$(arg altitude)-0.1-$(arg radius)}" />
-  <xacro:property name="mesh_file" value="package://ss_workshop/models/mesh/Plain_Cylinder.stl" />
+  <xacro:property name="mesh_file" value="package://ss_workshop/models/meshes/Plain_Cylinder.stl" />
   <!-- Macro for the inertia of a box -->
   <xacro:macro name="box_inertia" params="x y z mass">
@@ -33,5 +34,5 @@
 <link name="ring">
   <visual>
-    <origin xyz="0 0 0" rpy="0 0 0" />
+    <origin xyz="0 0 0" rpy="${pi/2} 0 0" />
     <geometry>
       <mesh filename="${mesh_file}" scale="${scale_r} ${scale_r} ${scale_t}" />
@@ -39,5 +40,5 @@
   </visual>
   <collision>
-    <origin xyz="0 0 0" rpy="${pi} 0 0" />
+    <origin xyz="0 0 0" rpy="${pi/2} 0 0" />
     <geometry>
       <mesh filename="${mesh_file}" scale="${scale_r} ${scale_r} ${scale_t}" />
@@ -49,3 +50,57 @@
   </inertial>
 </link>
+<link name="pillar">
+    <visual>
+      <geometry>
+        <cylinder length="${pillar_length}" radius="0.05"/>
+      </geometry>
+      <material name="blue">
+        <color rgba="0 0 0.8 1"/>
+      </material>
+    </visual>
+    <collision>
+      <geometry>
+        <cylinder length="${pillar_length}" radius="0.05"/>
+      </geometry>
+    </collision>
+    <inertial>
+      <mass value="10"/>
+      <xacro:cyl_inertia h="${pillar_length}" r="0.05" mass="10"/>
+    </inertial>
+</link>
+<link name="base">
+  <xacro:box_inertial x="0.5" y="0.5" z="0.05" mass="100">
+    <origin xyz="0 0 0" />
+  </xacro:box_inertial>
+  <visual>
+    <origin xyz="0 0 0" rpy="0 0 0" />
+    <geometry>
+      <box size="1 1 0.1"/>
+    </geometry>
+  </visual>
+  <collision>
+    <origin xyz="0 0 0" rpy="0 0 0" />
+    <geometry>
+      <box size="1 1 0.1"/>
+     </geometry>
+     <surface>
+        <friction>
+          <ode>
+            <mu>5000</mu>
+            <mu2>5000</mu2>
+          </ode>
+        </friction>
+      </surface>
+  </collision>
+</link>
+<joint name="${namespace}/base_to_pillar" type="fixed">
+  <origin xyz="0 0 ${(pillar_length/2) + 0.05}" rpy="0 0 0" />
+  <parent link="base" />
+  <child link="pillar" />
+</joint>
+<joint name="${namespace}/pillar_to_ring" type="fixed">
+  <origin xyz="0 0 ${$(arg radius) + (pillar_length/2)}" rpy="0 0 $(arg yaw)" />
+  <parent link="pillar" />
+  <child link="ring" />
+</joint>
 </robot>

File: models/urdf/pipe.xacro (robot description, xacro)
@@ -2,6 +2,7 @@
 <robot name="checkpoint" xmlns:xacro="http://ros.org/wiki/xacro">
   <xacro:arg name="mass" default="100" />
-  <xacro:arg name="radius" default="0.75" />
-  <xacro:arg name="thickness" default="0.05" />
+  <xacro:arg name="yaw" default="1.6" />
+  <xacro:arg name="radius" default="0.7" />
+  <xacro:arg name="thickness" default="5.0" />
   <xacro:arg name="altitude" default="1.5" />
   <xacro:property name="namespace" value="$(arg namespace)" />
@@ -10,5 +11,5 @@
   <xacro:property name="scale_t" value="${$(arg thickness)/50}" />
   <xacro:property name="pillar_length" value="${$(arg altitude)-0.1-$(arg radius)}" />
-  <xacro:property name="mesh_file" value="package://ss_workshop/models/mesh/Plain_Cylinder.stl" />
+  <xacro:property name="mesh_file" value="package://ss_workshop/models/meshes/Plain_Cylinder.stl" />
   <!-- Macro for the inertia of a box -->
   <xacro:macro name="box_inertia" params="x y z mass">
@@ -33,11 +34,14 @@
 <link name="ring">
   <visual>
-    <origin xyz="0 0 0" rpy="0 0 0" />
+    <origin xyz="0 0 0" rpy="${pi/2} 0 $(arg yaw)" />
     <geometry>
       <mesh filename="${mesh_file}" scale="${scale_r} ${scale_r} ${scale_t}" />
     </geometry>
+      <material name="blue">
+        <color rgba="0 0 0.8 1"/>
+      </material>
   </visual>
   <collision>
-    <origin xyz="0 0 0" rpy="${pi} 0 0" />
+    <origin xyz="0 0 0" rpy="${pi/2} 0 $(arg yaw)" />
     <geometry>
       <mesh filename="${mesh_file}" scale="${scale_r} ${scale_r} ${scale_t}" />
@@ -49,3 +53,56 @@
   </inertial>
 </link>
+<gazebo reference="ring">
+  <material>Gazebo/BlueTransparent</material>
+</gazebo>
+<!--
+<link name="pillar">
+    <visual>
+      <geometry>
+        <cylinder length="${pillar_length}" radius="0.05"/>
+      </geometry>
+      <material name="blue">
+        <color rgba="0 0 0.8 1"/>
+      </material>
+    </visual>
+    <collision>
+      <geometry>
+        <cylinder length="${pillar_length}" radius="0.05"/>
+      </geometry>
+    </collision>
+    <inertial>
+      <mass value="10"/>
+      <xacro:cyl_inertia h="${pillar_length}" r="0.05" mass="10"/>
+    </inertial>
+</link> -->
+<link name="base">
+  <xacro:box_inertial x="0.5" y="0.5" z="0.05" mass="100">
+    <origin xyz="0 0 0" />
+  </xacro:box_inertial>
+  <visual>
+    <origin xyz="0 0 0" rpy="0 0 $(arg yaw)" />
+    <geometry>
+      <box size="1 5 0.1"/>
+    </geometry>
+  </visual>
+  <collision>
+    <origin xyz="0 0 0" rpy="0 0 $(arg yaw)" />
+    <geometry>
+      <box size="1 1 0.1"/>
+     </geometry>
+     <surface>
+        <friction>
+          <ode>
+            <mu>5000</mu>
+            <mu2>5000</mu2>
+          </ode>
+        </friction>
+      </surface>
+  </collision>
+</link>
+<joint name="${namespace}/base_to_pipe" type="fixed">
+  <origin xyz="0 0 ${$(arg radius) + 0.05}" rpy="0 0 0" />
+  <parent link="base" />
+  <child link="ring" />
+</joint>
 </robot>
