Commit message: Lidar based avoidance added

File: models/urdf/pelican_laser.xacro (robot description, xacro)
@@ -177,5 +177,5 @@
   <!-- hokuyo -->
   <gazebo reference="hokuyo_link">
-    <sensor type="ray" name="head_hokuyo_sensor">
+    <sensor type="gpu_ray" name="head_hokuyo_sensor">
       <pose>0 0 0 0 0 0</pose>
       <visualize>false</visualize>
@@ -205,5 +205,5 @@
         </noise>
       </ray>
-      <plugin name="gazebo_ros_head_hokuyo_controller" filename="libgazebo_ros_laser.so">
+      <plugin name="gazebo_ros_head_hokuyo_controller" filename="libgazebo_ros_gpu_laser.so">
         <topicName>/rrbot/laser/scan</topicName>
         <frameName>hokuyo_link</frameName>

File: models/urdf/pelican_rod.xacro (robot description, xacro)
@@ -149,65 +149,45 @@
       izz="${0.5 * mass * (r*r)}" />
   </xacro:macro>
-  <!-- Hokuyo Laser -->
-  <link name="hokuyo_link">
+<link name="${namespace}/top_rod">
+    <visual>
+      <geometry>
+        <cylinder length="0.12" radius="0.02"/>
+      </geometry>
+    </visual>
     <collision>
-      <origin xyz="0 0 0" rpy="0 0 0"/>
       <geometry>
-    <box size="0.1 0.1 0.1"/>
+        <cylinder length="0.12" radius="0.05"/>
       </geometry>
     </collision>
+    <inertial>
+      <mass value="0.01"/>
+      <xacro:cyl_inertia h="0.12" r="0.05" mass="0.01"/>
+    </inertial>
+</link>
+<joint name="${namespace}/base_to_top_rod" type="fixed">
+  <origin xyz="0 0 0.12" rpy="0 0 0" />
+  <parent link="${namespace}/base_link" />
+  <child link="${namespace}/top_rod" />
+</joint>
+<link name="${namespace}/front_rod">
     <visual>
-      <origin xyz="0 0 0" rpy="0 0 0"/>
       <geometry>
-        <mesh filename="package://rrbot_description/meshes/hokuyo.dae"/>
+        <cylinder length="0.4" radius="0.01"/>
       </geometry>
     </visual>
+    <collision>
+      <geometry>
+        <cylinder length="0.4" radius="0.01"/>
+      </geometry>
+    </collision>
     <inertial>
-      <mass value="1e-5" />
-      <origin xyz="0 0 0" rpy="0 0 0"/>
-      <inertia ixx="1e-6" ixy="0" ixz="0" iyy="1e-6" iyz="0" izz="1e-6" />
+      <mass value="0.01"/>
+      <xacro:cyl_inertia h="0.4" r="0.01" mass="0.01"/>
     </inertial>
-  </link>
- <joint name="hokuyo_joint" type="fixed">
-    <axis xyz="0 1 0" />
-    <origin xyz="0 0 0.1" rpy="0 0 0"/>
-    <parent link="${namespace}/base_link"/>
-    <child link="hokuyo_link"/>
-  </joint>
-  <!-- hokuyo -->
-  <gazebo reference="hokuyo_link">
-    <sensor type="ray" name="head_hokuyo_sensor">
-      <pose>0 0 0 0 0 0</pose>
-      <visualize>false</visualize>
-      <update_rate>40</update_rate>
-      <ray>
-        <scan>
-          <horizontal>
-            <samples>720</samples>
-            <resolution>1</resolution>
-            <min_angle>-1.570796</min_angle>
-            <max_angle>1.570796</max_angle>
-          </horizontal>
-        </scan>
-        <range>
-          <min>0.10</min>
-          <max>30.0</max>
-          <resolution>0.01</resolution>
-        </range>
-        <noise>
-          <type>gaussian</type>
-          <!-- Noise parameters based on published spec for Hokuyo laser
-               achieving "+-30mm" accuracy at range < 10m.  A mean of 0.0m and
-               stddev of 0.01m will put 99.7% of samples within 0.03m of the true
-               reading. -->
-          <mean>0.0</mean>
-          <stddev>0.01</stddev>
-        </noise>
-      </ray>
-      <plugin name="gazebo_ros_head_hokuyo_controller" filename="libgazebo_ros_laser.so">
-        <topicName>/rrbot/laser/scan</topicName>
-        <frameName>hokuyo_link</frameName>
-      </plugin>
-    </sensor>
-  </gazebo>
+</link>
+<joint name="${namespace}/top_to_front_rod" type="fixed">
+  <origin xyz="0.2 0 0.05" rpy="0 ${pi/2} 0" />
+  <parent link="${namespace}/top_rod" />
+  <child link="${namespace}/front_rod" />
+</joint>
 </robot>

File: models/urdf/pipe.xacro (robot description, xacro)
@@ -3,5 +3,5 @@
   <xacro:arg name="mass" default="100" />
   <xacro:arg name="yaw" default="1.6" />
-  <xacro:arg name="radius" default="0.5" />
+  <xacro:arg name="radius" default="1.2" />
   <xacro:arg name="thickness" default="5.0" />
   <xacro:arg name="altitude" default="1.5" />
